File: Hardware/ChargeControl/ChargeControl.sch (KiCad schematic (older format))
At the start: 28 parts, among them J1 Conn_01x03, J2 Conn_01x04, J3 Conn_01x04, J4 Conn_01x08, Q1 Q-FET-N-SSM3K36MFV, U1 74LVC1G14, U2 MCP602

Commit message: Older PCB updates
Parts:
- added R13: 3.3k, Resistor_SMD:R_0603_1608Metric_Pad1.05x0.95mm_HandSolder, symbol Device:R
- added R14: 100k, Resistor_SMD:R_0603_1608Metric_Pad1.05x0.95mm_HandSolder, symbol Device:R
- added TP1, TP10, TP11, TP12, TP13, TP14, TP15, TP16, TP17, TP18, TP19, TP2, TP3, TP4, TP5, TP6, TP7, TP8, TP9: TestPoint, TestPoint:TestPoint_Loop_D2.50mm_Drill1.0mm_LowProfile, symbol Connector:TestPoint
- U2: footprint Package_SO:MSOP-8_3x3mm_P0.65mm -> Package_SO:SOIC-8_3.9x4.9mm_P1.27mm
Connections:
- net +12V: now also TP19.1
- net +3V3: now also TP14.1
- net 1.4V: now also TP17.1
- net 13V8_FROM_CHARGER: now also TP7.1
- net 2.2V: now also TP16.1
- net CHARGER_POWER_SENSE: now also TP8.1
- net GND: now also R14.2, TP15.1
- net GNDPWR: now also TP18.1
- net PILOT_EV_CHARGE: now also R13.1, TP2.1; no longer Q1.1 (G)
- net PILOT_OUT: now also TP9.1
- net PLUG_PILOT: now also TP1.1
- net PLUG_PROXIMITY: now also TP5.1
- net PROXIMITY_0: now also TP13.1
- net PROXIMITY_1: now also TP12.1
- net at R2.1, R3.2, U1.2: now also TP6.1
- net at D1.3 (C), R1.2, R2.2: now also TP4.1
- net at R8.2, U2.2 (-): now also TP10.1
- net at R9.2, U2.6 (-): now also TP11.1
- new net: Q1.1 (G), R13.2, R14.1, TP3.1
