File: Hardware/Contactor Control/Contactor Control.sch (KiCad schematic (older format))
At the start: 16 parts, among them J1 Conn_01x02, J2 Conn_01x02, J3 Conn_01x01, J4 Conn_02x02_Top_Bottom, Q1 Q-FET-N-PMN20EN

Commit message: Older PCB updates
Other:
- note added: "Problems with transistor failure. 2021-01-24.\nHypothesis: \n\nFirst time:\nground for control signal and 12V not connected when testing, causing too high gate voltage?\n\nSecond time:\npins 1 & 2 to contactor shorted when troublshooting, causing too high current through transistor. \n\nCould protect against second case with a resistor? Max current is 6.7A, resistance of 1.8 Ohm would do it. Uncl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"
Changed lines of the file:
@@
 EESchema Schematic File Version 4
-LIBS:Contractor Control-cache
+LIBS:Contactor Control-cache
 EELAYER 30 0
 EELAYER END
@@
 	1    0    0    -1
 $EndComp
+Text Notes 5800 2900 0    50   ~ 0
+Problems with transistor failure. 2021-01-24.\nHypothesis: \n\nFirst time:\nground for control signal and 12V not connected when testing, causing too high gate voltage?\n\nSecond time:\npins 1 & 2 to contactor shorted when troublshooting, causing too high current through transistor. \n\nCould protect against second case with a resistor? Max current is 6.7A, resistance of 1.8 Ohm would do it. Unclear if it would prevent contactor operation.\n\nAlso, replaced R2 with 30 kOhm.\n\nReplace the transistor again for now.\n
 $EndSCHEMATC
