File: Hardware/DCDC Power Control/Microcontroller.sch (KiCad schematic (older format))
At the start: 20 parts, among them J6 Conn_01x03_Female, U2 NCP785AH33T1G, U3 ATtiny414-SS

Commit message: Older PCB updates
Parts:
- removed J6: Conn_01x03_Female, Connector_PinSocket_2.54mm:PinSocket_1x03_P2.54mm_Vertical, symbol Connector:Conn_01x03_Female
- added D3: LED, LED_SMD:LED_0603_1608Metric_Castellated, symbol Device:LED
- added J6: Conn_01x04_Female, Connector_PinSocket_2.54mm:PinSocket_1x04_P2.54mm_Vertical, symbol Connector:Conn_01x04_Female
- added J7: Conn_01x02, Connector_PinHeader_2.54mm:PinHeader_1x02_P2.54mm_Vertical, symbol Connector_Generic:Conn_01x02
- added R29: ?, Resistor_SMD:R_0603_1608Metric_Pad1.05x0.95mm_HandSolder, symbol Device:R
- C1, C4: footprint Capacitor_SMD:C_0805_2012Metric_Pad1.15x1.40mm_HandSolder -> Capacitor_SMD:C_0603_1608Metric_Pad1.05x0.95mm_HandSolder
Connections:
- net +3V3: now also J6.3 (Pin_3)
- net DCDC_PRECHARGE_GATE: now also U3.11 (PA1); no longer U3.13 (PA3)
- net GNDPWR: now also J6.2 (Pin_2), R29.2
- net UDPI: now also J6.1 (Pin_1)
- net PB3: now reaches U3.6 (PB3)
- net PB3: now also D3.2 (A), J7.2 (Pin_2)
- net PB2: now reaches U3.7 (PB2)
- net PB2: now also J7.1 (Pin_1)
- new net: D3.1 (K), R29.1
- new net PA3: J6.4 (Pin_4), U3.13 (PA3)
Changed lines of the file:
@@
 Wire Wire Line
 	5600 3350 5800 3350
-Text HLabel 5800 3350 2    50   Output ~ 0
+Text HLabel 5800 3150 2    50   Output ~ 0
 DCDC_PRECHARGE_GATE
-Text HLabel 1800 3050 0    50   Input ~ 0
+Text HLabel 1550 3250 0    50   Input ~ 0
 SWITCH_A
 Text HLabel 5800 3250 2    50   Input ~ 0
@@
 L power:GNDPWR #PWR011
 U 1 1 60252462
-P 1900 3150
-F 0 "#PWR011" H 1900 2950 50  0001 C CNN
-F 1 "GNDPWR" H 1904 2996 50  0000 C CNN
-F 2 "" H 1900 3100 50  0001 C CNN
-F 3 "" H 1900 3100 50  0001 C CNN
-	1    1900 3150
-	1    0    0    -1
-$EndComp
-Wire Wire Line
-	1800 3050 1900 3050
-Wire Wire Line
-	1900 3050 1900 3150
+P 1650 3350
+F 0 "#PWR011" H 1650 3150 50  0001 C CNN
+F 1 "GNDPWR" H 1654 3196 50  0000 C CNN
+F 2 "" H 1650 3300 50  0001 C CNN
+F 3 "" H 1650 3300 50  0001 C CNN
+	1    1650 3350
+	1    0    0    -1
+$EndComp
+Wire Wire Line
+	1550 3250 1650 3250
+Wire Wire Line
+	1650 3250 1650 3350
 Wire Wire Line
 	5800 3650 5600 3650
@@
 F 0 "C1" H 2065 5196 50  0000 L CNN
 F 1 "100 nF/3.3V" H 2065 5105 50  0000 L CNN
-F 2 "Capacitor_SMD:C_0805_2012Metric_Pad1.15x1.40mm_HandSolder" H 1988 5000 50  0001 C CNN
+F 2 "Capacitor_SMD:C_0603_1608Metric_Pad1.05x0.95mm_HandSolder" H 1988 5000 50  0001 C CNN
 F 3 "~" H 1950 5150 50  0001 C CNN
 F 4 "CL21X226MRQNNNE" H 1950 5150 50  0001 C CNN "PN"
@@
 F 0 "C4" H 3415 4346 50  0000 L CNN
 F 1 "100 nF/3.3V" H 3415 4255 50  0000 L CNN
-F 2 "Capacitor_SMD:C_0805_2012Metric_Pad1.15x1.40mm_HandSolder" H 3338 4150 50  0001 C CNN
+F 2 "Capacitor_SMD:C_0603_1608Metric_Pad1.05x0.95mm_HandSolder" H 3338 4150 50  0001 C CNN
 F 3 "~" H 3300 4300 50  0001 C CNN
 F 4 "CL21X226MRQNNNE" H 3300 4300 50  0001 C CNN "PN"
@@
 L power:GNDPWR #PWR0101
 U 1 1 602BE7C7
-P 1750 2750
-F 0 "#PWR0101" H 1750 2550 50  0001 C CNN
-F 1 "GNDPWR" H 1754 2596 50  0000 C CNN
-F 2 "" H 1750 2700 50  0001 C CNN
-F 3 "" H 1750 2700 50  0001 C CNN
-	1    1750 2750
-	1    0    0    -1
-$EndComp
-Wire Wire Line
-	1600 2700 1750 2700
-Wire Wire Line
-	1750 2700 1750 2750
-Wire Wire Line
-	1600 2600 1900 2600
-Text Label 1900 2600 0    50   ~ 0
+P 2050 2750
+F 0 "#PWR0101" H 2050 2550 50  0001 C CNN
+F 1 "GNDPWR" H 2054 2596 50  0000 C CNN
+F 2 "" H 2050 2700 50  0001 C CNN
+F 3 "" H 2050 2700 50  0001 C CNN
+	1    2050 2750
+	1    0    0    -1
+$EndComp
+Wire Wire Line
+	1600 2700 2050 2700
+Wire Wire Line
+	2050 2700 2050 2750
+Wire Wire Line
+	1600 2600 1950 2600
+Text Label 1650 2800 0    50   ~ 0
 UDPI
 $Comp
@@
 	4150 2050 4150 2200
 $Comp
-L Connector:Conn_01x03_Female J6
-U 1 1 602C7DFB
-P 1400 2600
-F 0 "J6" H 1292 2275 50  0000 C CNN
-F 1 "Conn_01x03_Female" H 1292 2366 50  0000 C CNN
-F 2 "Connector_PinSocket_2.54mm:PinSocket_1x03_P2.54mm_Vertical" H 1400 2600 50  0001 C CNN
-F 3 "~" H 1400 2600 50  0001 C CNN
-	1    1400 2600
-	-1   0    0    1
-$EndComp
-$Comp
 L power:+3.3V #PWR0104
 U 1 1 602CDFD0
@@
 $EndComp
 Wire Wire Line
-	1600 2500 1950 2500
-Wire Wire Line
-	1950 2500 1950 2400
+	1950 2600 1950 2400
 Wire Wire Line
 	5600 3750 5850 3750
 Wire Wire Line
 	4400 3050 4200 3050
+Wire Wire Line
+	5600 3150 5800 3150
+Wire Wire Line
+	4400 3250 4200 3250
+Wire Wire Line
+	4400 3350 4200 3350
+Text Label 5800 3350 0    50   ~ 0
+PA3
+Text Label 4200 3250 2    50   ~ 0
+PB2
+Text Label 4200 3350 2    50   ~ 0
+PB3
+Wire Wire Line
+	6900 4700 6800 4700
+Text Label 6800 4600 2    50   ~ 0
+PB2
+Text Label 6800 4700 2    50   ~ 0
+PB3
+Text Label 5400 5000 2    50   ~ 0
+PB3
+$Comp
+L Device:LED D3
+U 1 1 601FA510
+P 5600 5200
+F 0 "D3" V 5639 5083 50  0000 R CNN
+F 1 "LED" V 5548 5083 50  0000 R CNN
+F 2 "LED_SMD:LED_0603_1608Metric_Castellated" H 5600 5200 50  0001 C CNN
+F 3 "~" H 5600 5200 50  0001 C CNN
+	1    5600 5200
+	0    -1   -1   0
+$EndComp
+Wire Wire Line
+	5400 5000 5600 5000
+Wire Wire Line
+	5600 5000 5600 5050
+$Comp
+L Device:R R29
+U 1 1 601FD74E
+P 5600 5600
+F 0 "R29" H 5670 5646 50  0000 L CNN
+F 1 "?" H 5670 5555 50  0000 L CNN
+F 2 "Resistor_SMD:R_0603_1608Metric_Pad1.05x0.95mm_HandSolder" V 5530 5600 50  0001 C CNN
+F 3 "~" H 5600 5600 50  0001 C CNN
+	1    5600 5600
+	1    0    0    -1
+$EndComp
+Wire Wire Line
+	5600 5450 5600 5350
+$Comp
+L power:GNDPWR #PWR0105
+U 1 1 601FF656
+P 5600 5850
+F 0 "#PWR0105" H 5600 5650 50  0001 C CNN
+F 1 "GNDPWR" H 5604 5696 50  0000 C CNN
+F 2 "" H 5600 5800 50  0001 C CNN
+F 3 "" H 5600 5800 50  0001 C CNN
+	1    5600 5850
+	1    0    0    -1
+$EndComp
+Wire Wire Line
+	5600 5850 5600 5750
+$Comp
+L Connector:Conn_01x04_Female J6
+U 1 1 60237804
+P 1400 2700
+F 0 "J6" H 1292 2275 50  0000 C CNN
+F 1 "Conn_01x04_Female" H 1292 2366 50  0000 C CNN
+F 2 "Connector_PinSocket_2.54mm:PinSocket_1x04_P2.54mm_Vertical" H 1400 2700 50  0001 C CNN
+F 3 "~" H 1400 2700 50  0001 C CNN
+	1    1400 2700
+	-1   0    0    1
+$EndComp
+Wire Wire Line
+	1600 2800 1650 2800
+Text Label 1800 2500 0    50   ~ 0
+PA3
+Wire Wire Line
+	1800 2500 1600 2500
+$Comp
+L Connector_Generic:Conn_01x02 J7
+U 1 1 6026B5C6
+P 7100 4600
+F 0 "J7" H 7180 4592 50  0000 L CNN
+F 1 "Conn_01x02" H 7180 4501 50  0000 L CNN
+F 2 "Connector_PinHeader_2.54mm:PinHeader_1x02_P2.54mm_Vertical" H 7100 4600 50  0001 C CNN
+F 3 "~" H 7100 4600 50  0001 C CNN
+	1    7100 4600
+	1    0    0    -1
+$EndComp
+Wire Wire Line
+	6800 4600 6900 4600
 $EndSCHEMATC
