File: Hardware/DCDC Power Control/power_switches.sch (KiCad schematic (older format))
At the start: 33 parts, among them Q1 BSS123, Q2 MCT06P10, Q3 BSS123, Q4 MCT06P10, Q5 BSS123, Q6 SQJ479EP-T1_GE3

Commit message: Older PCB updates
Parts:
- Q6: footprint Package_SO:Vishay_PowerPAK_1212-8_Single -> erland-footprints:Q-VISHAY-PowerPAK SO-8L Single
Changed lines of the file:
@@
 F 0 "Q6" V 7242 3600 50  0000 C CNN
 F 1 "SQJ479EP-T1_GE3" V 7151 3600 50  0000 C CNN
-F 2 "Package_SO:Vishay_PowerPAK_1212-8_Single" H 7100 3525 50  0001 L CIN
+F 2 "erland-footprints:Q-VISHAY-PowerPAK SO-8L Single" H 7100 3525 50  0001 L CIN
 F 3 "https://www.vishay.com/docs/75129/sqj479ep.pdf" V 6900 3600 50  0001 L CNN
 	1    6900 3600
